File: circuit/usbkey.brd (EAGLE design)
At the start: 69 x 95 mm, 12 parts, among them IC1 ATmega168P, Q1 16MHz, X2 USB

Commit message: fix
Parts:
- added C4: 0.1u, c-j:50-0302-2.54
- R1, R2: value 168 -> 68
Connections:
- net GND: now also C4.PAD1
- net N$9: now also C4.PAD2
Changed lines of the file:
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@@
 <attribute name="VALUE" x="22.352" y="30.353" size="1.27" layer="27" ratio="10"/>
 </element>
-<element name="R1" library="r-j" package="1/4W-7.62H" value="168" x="29.21" y="38.1" smashed="yes">
+<element name="R1" library="r-j" package="1/4W-7.62H" value="68" x="29.21" y="38.1" smashed="yes">
 <attribute name="NAME" x="27.0764" y="35.4584" size="1.27" layer="25" ratio="10"/>
 <attribute name="VALUE" x="27.0764" y="35.7886" size="1.27" layer="27" ratio="10"/>
 </element>
-<element name="R2" library="r-j" package="1/4W-7.62H" value="168" x="29.21" y="40.64"/>
+<element name="R2" library="r-j" package="1/4W-7.62H" value="68" x="29.21" y="40.64"/>
 <element name="R3" library="r-j" package="1/4W-2.54V" value="1.5k" x="17.78" y="38.1" smashed="yes" rot="R270">
 <attribute name="NAME" x="17.018" y="35.0774" size="0.9906" layer="25" ratio="10"/>
 <attribute name="VALUE" x="17.2974" y="39.7256" size="0.9906" layer="27" ratio="10" rot="R270"/>
 </element>
+<element name="C4" library="c-j" package="50-0302-2.54" value="0.1u" x="-2.54" y="-13.97"/>
 </elements>
 <signals>
@@
 <wire x1="53.34" y1="15.24" x2="53.34" y2="7.62" width="0.8128" layer="16"/>
 <wire x1="2.54" y1="22.86" x2="22.86" y2="22.86" width="0.8128" layer="16"/>
+<contactref element="C4" pad="PAD1"/>
 <wire x1="50.8" y1="2.54" x2="53.34" y2="7.62" width="0" layer="19" extent="16-16"/>
+<wire x1="-3.81" y1="-13.97" x2="2.54" y2="22.86" width="0" layer="19" extent="16-16"/>
 </signal>
 <signal name="N$2">
@@
 <via x="53.34" y="17.78" extent="1-16" drill="0.8"/>
 <wire x1="53.34" y1="17.78" x2="55.88" y2="17.78" width="0.8128" layer="16"/>
+<contactref element="C4" pad="PAD2"/>
+<wire x1="-1.27" y1="-13.97" x2="40.64" y2="12.7" width="0" layer="19" extent="1-1"/>
 </signal>
 <signal name="N$10">
